Commit message: spot loads in bullet! gets warning that base_footprint has no inertia but that's for Gazebo Compatibility. Easy fix is to simply remove it from resultant urdf

File: bullet/src/spotmicro/util/pybullet_data/assets/urdf/spot.urdf (robot description, URDF)
Before this commit: robot spot, 23 links, 22 joints
Links:
- added link base_footprint
- link base_link: mass 2.80 -> 2.8
- link chassis_front_link: mass 0.20 -> 0.2
- link chassis_rear_link: mass 0.20 -> 0.2
- link front_left_foot_link: geometry collision box size=0.026 0.02 0.115; visual mesh filename=stl/lfoot.stl scale=0.001 0.001 0.001
- link front_left_leg_link_cover: mass None -> 0.05; geometry collision box size=0.028 0.036 0.12; visual mesh filename=stl/larm_cover.stl scale=0.001 0.001 0.001
- link front_left_shoulder_link: mass 0.10 -> 0.1
- link front_right_foot_link: geometry collision box size=0.026 0.02 0.115; visual mesh filename=stl/rfoot.stl scale=0.001 0.001 0.001
- link front_right_leg_link_cover: mass None -> 0.05; geometry collision box size=0.028 0.036 0.12; visual mesh filename=stl/rarm_cover.stl scale=0.001 0.001 0.001
- link front_right_shoulder_link: mass 0.10 -> 0.1
- link rear_left_foot_link: geometry collision box size=0.026 0.02 0.115; visual mesh filename=stl/lfoot.stl scale=0.001 0.001 0.001
- link rear_left_leg_link_cover: mass None -> 0.05; geometry collision box size=0.028 0.036 0.12; visual mesh filename=stl/larm_cover.stl scale=0.001 0.001 0.001
- link rear_left_shoulder_link: mass 0.10 -> 0.1
- link rear_right_foot_link: geometry collision box size=0.026 0.02 0.115; visual mesh filename=stl/rfoot.stl scale=0.001 0.001 0.001
- link rear_right_leg_link_cover: mass None -> 0.05; geometry collision box size=0.028 0.036 0.12; visual mesh filename=stl/rarm_cover.stl scale=0.001 0.001 0.001
- link rear_right_shoulder_link: mass 0.10 -> 0.1
Joints:
- added joint base_base: type fixed, parent base_footprint, child base_link, origin xyz=0 0 0 rpy=0 0 0
- joint chassis_base_front: origin (none) -> xyz=0 0 0 rpy=0 0 0
- joint chassis_base_rear: origin (none) -> xyz=0 0 0 rpy=0 0 0
- joint foot_motor_front_left: limit lower=-0.1 upper=2.59 effort=1000.0 velocity=0.5 -> lower=-0.1 upper=2.59 effort=3.53 velocity=9.52
- joint foot_motor_front_right: limit lower=-0.1 upper=2.59 effort=1000.0 velocity=0.5 -> lower=-0.1 upper=2.59 effort=3.53 velocity=9.52
- joint foot_motor_rear_left: limit lower=-0.1 upper=2.59 effort=1000.0 velocity=0.5 -> lower=-0.1 upper=2.59 effort=3.53 velocity=9.52
- joint foot_motor_rear_right: limit lower=-0.1 upper=2.59 effort=1000.0 velocity=0.5 -> lower=-0.1 upper=2.59 effort=3.53 velocity=9.52
- joint front_left_leg_cover_joint: origin xyz=0 0 0 -> xyz=0 0 0 rpy=0 0 0
- joint front_left_toe: origin xyz=0 0 -0.115 -> xyz=0 0 -0.115 rpy=0 0 0
- joint front_right_leg_cover_joint: origin xyz=0 0 0 -> xyz=0 0 0 rpy=0 0 0
- joint front_right_toe: origin xyz=0 0 -0.115 -> xyz=0 0 -0.115 rpy=0 0 0
- joint motor_front_left_leg: limit lower=-2.666 upper=1.548 effort=1000.0 velocity=0.5 -> lower=-2.17 upper=0.97 effort=3.53 velocity=9.52
- joint motor_front_left_shoulder: limit lower=-0.548 upper=0.548 effort=1000.0 velocity=0.7 -> lower=-0.548 upper=0.548 effort=3.53 velocity=9.52
- joint motor_front_right_leg: limit lower=-2.666 upper=1.548 effort=1000.0 velocity=0.5 -> lower=-2.17 upper=0.97 effort=3.53 velocity=9.52
- joint motor_front_right_shoulder: limit lower=-0.548 upper=0.548 effort=1000.0 velocity=0.7 -> lower=-0.548 upper=0.548 effort=3.53 velocity=9.52
- joint motor_rear_left_leg: limit lower=-2.666 upper=1.548 effort=1000.0 velocity=0.5 -> lower=-2.17 upper=0.97 effort=3.53 velocity=9.52
- joint motor_rear_left_shoulder: limit lower=-0.548 upper=0.548 effort=1000.0 velocity=0.7 -> lower=-0.548 upper=0.548 effort=3.53 velocity=9.52
- joint motor_rear_right_leg: limit lower=-2.666 upper=1.548 effort=1000.0 velocity=0.5 -> lower=-2.17 upper=0.97 effort=3.53 velocity=9.52
- joint motor_rear_right_shoulder: limit lower=-0.548 upper=0.548 effort=1000.0 velocity=0.7 -> lower=-0.548 upper=0.548 effort=3.53 velocity=9.52
- joint rear_left_leg_cover_joint: origin xyz=0 0 0 -> xyz=0 0 0 rpy=0 0 0
- joint rear_left_toe: origin xyz=0 0 -0.115 -> xyz=0 0 -0.115 rpy=0 0 0
- joint rear_right_leg_cover_joint: origin xyz=0 0 0 -> xyz=0 0 0 rpy=0 0 0
- joint rear_right_toe: origin xyz=0 0 -0.115 -> xyz=0 0 -0.115 rpy=0 0 0

Commit message: added kinematics package for Spot. writing test script now

File: bullet/src/spotmicro/util/pybullet_data/assets/urdf/spot.urdf (robot description, URDF)
Before this commit: robot spot, 24 links, 23 joints
Links:
- removed link base_footprint
Joints:
- removed joint base_base

Commit message: IK works. The problem was the URDF and Motor model.. need to fix those

File: bullet/src/spotmicro/util/pybullet_data/assets/urdf/spot.urdf (robot description, URDF)
Before this commit: robot spot, 23 links, 22 joints
Links:
- link base_link: mass 2.8 -> 2.80
- link chassis_front_link: mass 0.2 -> 0.20
- link chassis_rear_link: mass 0.2 -> 0.20
- link front_left_foot_link: geometry collision box size=0.026 0.020 0.115; visual mesh filename=stl/lfoot.stl scale=0.001 0.001 0.001
- link front_left_leg_link_cover: mass 0.05 -> None; geometry visual mesh filename=stl/larm_cover.stl scale=0.001 0.001 0.001
- link front_left_shoulder_link: mass 0.1 -> 0.10
- link front_right_foot_link: geometry collision box size=0.026 0.020 0.115; visual mesh filename=stl/rfoot.stl scale=0.001 0.001 0.001
- link front_right_leg_link_cover: mass 0.05 -> None; geometry visual mesh filename=stl/rarm_cover.stl scale=0.001 0.001 0.001
- link front_right_shoulder_link: mass 0.1 -> 0.10
- link rear_left_foot_link: geometry collision box size=0.026 0.020 0.115; visual mesh filename=stl/lfoot.stl scale=0.001 0.001 0.001
- link rear_left_leg_link_cover: mass 0.05 -> None; geometry visual mesh filename=stl/larm_cover.stl scale=0.001 0.001 0.001
- link rear_left_shoulder_link: mass 0.1 -> 0.10
- link rear_right_foot_link: geometry collision box size=0.026 0.020 0.115; visual mesh filename=stl/rfoot.stl scale=0.001 0.001 0.001
- link rear_right_leg_link_cover: mass 0.05 -> None; geometry visual mesh filename=stl/rarm_cover.stl scale=0.001 0.001 0.001
- link rear_right_shoulder_link: mass 0.1 -> 0.10
Joints:
- joint chassis_base_front: origin xyz=0 0 0 rpy=0 0 0 -> (none)
- joint chassis_base_rear: origin xyz=0 0 0 rpy=0 0 0 -> (none)
- joint foot_motor_front_left: limit lower=-0.1 upper=2.59 effort=3.53 velocity=9.52 -> lower=-0.1 upper=2.59 effort=1000.0 velocity=0.5
- joint foot_motor_front_right: limit lower=-0.1 upper=2.59 effort=3.53 velocity=9.52 -> lower=-0.1 upper=2.59 effort=1000.0 velocity=0.5
- joint foot_motor_rear_left: limit lower=-0.1 upper=2.59 effort=3.53 velocity=9.52 -> lower=-0.1 upper=2.59 effort=1000.0 velocity=0.5
- joint foot_motor_rear_right: limit lower=-0.1 upper=2.59 effort=3.53 velocity=9.52 -> lower=-0.1 upper=2.59 effort=1000.0 velocity=0.5
- joint front_left_leg_cover_joint: origin xyz=0 0 0 rpy=0 0 0 -> xyz=0 0 0
- joint front_left_toe: origin xyz=0 0 -0.115 rpy=0 0 0 -> xyz=0 0 -0.115
- joint front_right_leg_cover_joint: origin xyz=0 0 0 rpy=0 0 0 -> xyz=0 0 0
- joint front_right_toe: origin xyz=0 0 -0.115 rpy=0 0 0 -> xyz=0 0 -0.115
- joint motor_front_left_leg: limit lower=-2.17 upper=0.97 effort=3.53 velocity=9.52 -> lower=-2.666 upper=1.548 effort=1000.0 velocity=0.5
- joint motor_front_left_shoulder: limit lower=-0.548 upper=0.548 effort=3.53 velocity=9.52 -> lower=-0.548 upper=0.548 effort=1000.0 velocity=0.7
- joint motor_front_right_leg: limit lower=-2.17 upper=0.97 effort=3.53 velocity=9.52 -> lower=-2.666 upper=1.548 effort=1000.0 velocity=0.5
- joint motor_front_right_shoulder: limit lower=-0.548 upper=0.548 effort=3.53 velocity=9.52 -> lower=-0.548 upper=0.548 effort=1000.0 velocity=0.7
- joint motor_rear_left_leg: limit lower=-2.17 upper=0.97 effort=3.53 velocity=9.52 -> lower=-2.666 upper=1.548 effort=1000.0 velocity=0.5
- joint motor_rear_left_shoulder: limit lower=-0.548 upper=0.548 effort=3.53 velocity=9.52 -> lower=-0.548 upper=0.548 effort=1000.0 velocity=0.7
- joint motor_rear_right_leg: limit lower=-2.17 upper=0.97 effort=3.53 velocity=9.52 -> lower=-2.666 upper=1.548 effort=1000.0 velocity=0.5
- joint motor_rear_right_shoulder: limit lower=-0.548 upper=0.548 effort=3.53 velocity=9.52 -> lower=-0.548 upper=0.548 effort=1000.0 velocity=0.7
- joint rear_left_leg_cover_joint: origin xyz=0 0 0 rpy=0 0 0 -> xyz=0 0 0
- joint rear_left_toe: origin xyz=0 0 -0.115 rpy=0 0 0 -> xyz=0 0 -0.115
- joint rear_right_leg_cover_joint: origin xyz=0 0 0 rpy=0 0 0 -> xyz=0 0 0
- joint rear_right_toe: origin xyz=0 0 -0.115 rpy=0 0 0 -> xyz=0 0 -0.115

File: mini_ros/urdf/spot.urdf.xacro (robot description, xacro)
@@ -10,5 +10,5 @@
               origin_rpy="0 0 0" origin_xyz="-0.045 -0.060 -0.015"
               i_rpy="0 0 0" i_xyz="0 0 0"
-              mass="2.8"
+              mass="1.2"
               c_xyz="0 0 0"
               length="0.14"
@@ -22,5 +22,5 @@
               origin_rpy="0 0 0" origin_xyz="-0.040 -0.060 -0.0140"
               i_rpy="0 0 0" i_xyz="-0.145 0 0"
-              mass="0.2"
+              mass="0.05"
               c_xyz="-0.145 0 0"
               length="0.058"
@@ -34,5 +34,5 @@
               origin_rpy="0 0 0" origin_xyz="-0.040 -0.060 -0.0140"
               i_rpy="0 0 0" i_xyz="0.135 0 0"
-              mass="0.2"
+              mass="0.05"
               c_xyz="0.135 0 0"
               length="0.04"
@@ -47,5 +47,5 @@
               origin_rpy="0 0 0" origin_xyz="-0.135 -0.02 -0.01"
               i_rpy="0 0 0" i_xyz="0 0 0"
-              mass="0.1"
+              mass="0.075"
               c_xyz="0 0 0"
               length="0.044"
@@ -59,5 +59,5 @@
               origin_rpy="0 0 0" origin_xyz="-0.125 0.04 -0.02"
               i_rpy="0 0 0" i_xyz="0.0 0.0 -0.050"
-              mass="0.05"
+              mass="0.005"
               c_xyz="0.0 0.0 -0.050"
               length="0.028"
@@ -71,5 +71,5 @@
               origin_rpy="0 0 0" origin_xyz="-0.125 0.04 -0.02"
               i_rpy="0 0 0" i_xyz="0.0 0.0 -0.050"
-              mass="0.15"
+              mass="0.08"
               c_xyz="0.0 0.0 -0.050"
               length="0.028"
@@ -83,5 +83,5 @@
               origin_rpy="0 0 0" origin_xyz="-0.120 0.04 0.1"
               i_rpy="0 0 0" i_xyz="0.0 0.0 -0.050"
-              mass="0.1"
+              mass="0.034"
               c_xyz="0.0 0.0 -0.050"
               length="0.026"
@@ -95,5 +95,5 @@
               origin_rpy="0 -0.40010 0" origin_xyz="0 -0.01 0"
               i_rpy="0 0 0" i_xyz="0 0 0"
-              mass="0.05"
+              mass="0.0044"
               c_xyz="0 0 0"
               length="0.02"
@@ -109,5 +109,5 @@
               origin_rpy="0 0 0" origin_xyz="-0.135 -0.09 -0.01"
               i_rpy="0 0 0" i_xyz="0 0 0"
-              mass="0.1"
+              mass="0.075"
               c_xyz="0 0 0"
               length="0.044"
@@ -121,5 +121,5 @@
               origin_rpy="0 0 0" origin_xyz="-0.125 -0.15 -0.02"
               i_rpy="0 0 0" i_xyz="0.0 0.0 -0.050"
-              mass="0.05"
+              mass="0.005"
               c_xyz="0.0 0.0 -0.050"
               length="0.028"
@@ -133,5 +133,5 @@
               origin_rpy="0 0 0" origin_xyz="-0.125 -0.15 -0.02"
               i_rpy="0 0 0" i_xyz="0.0 0.0 -0.050"
-              mass="0.15"
+              mass="0.08"
               c_xyz="0.0 0.0 -0.050"
               length="0.028"
@@ -145,5 +145,5 @@
               origin_rpy="0 0 0" origin_xyz="-0.120 -0.15 0.1"
               i_rpy="0 0 0" i_xyz="0.0 0.0 -0.050"
-              mass="0.1"
+              mass="0.034"
               c_xyz="0.0 0.0 -0.050"
               length="0.026"
@@ -157,5 +157,5 @@
               origin_rpy="0 -0.40010 0" origin_xyz="0 -0.01 0"
               i_rpy="0 0 0" i_xyz="0 0 0"
-              mass="0.05"
+              mass="0.0044"
               c_xyz="0 0 0"
               length="0.02"
@@ -171,5 +171,5 @@
               origin_rpy="0 0 0" origin_xyz="-0.135 -0.02 -0.01"
               i_rpy="0 0 0" i_xyz="0 0 0"
-              mass="0.1"
+              mass="0.075"
               c_xyz="0 0 0"
               length="0.044"
@@ -183,5 +183,5 @@
               origin_rpy="0 0 0" origin_xyz="-0.125 0.04 -0.02"
               i_rpy="0 0 0" i_xyz="0.0 0.0 -0.050"
-              mass="0.05"
+              mass="0.005"
               c_xyz="0.0 0.0 -0.050"
               length="0.028"
@@ -195,5 +195,5 @@
               origin_rpy="0 0 0" origin_xyz="-0.125 0.04 -0.02"
               i_rpy="0 0 0" i_xyz="0.0 0.0 -0.050"
-              mass="0.15"
+              mass="0.08"
               c_xyz="0.0 0.0 -0.050"
               length="0.028"
@@ -207,5 +207,5 @@
               origin_rpy="0 0 0" origin_xyz="-0.120 0.04 0.1"
               i_rpy="0 0 0" i_xyz="0.0 0.0 -0.050"
-              mass="0.1"
+              mass="0.034"
               c_xyz="0.0 0.0 -0.050"
               length="0.026"
@@ -219,5 +219,5 @@
               origin_rpy="0 -0.40010 0" origin_xyz="0 -0.01 0"
               i_rpy="0 0 0" i_xyz="0 0 0"
-              mass="0.05"
+              mass="0.0044"
               c_xyz="0 0 0"
               length="0.02"
@@ -233,5 +233,5 @@
               origin_rpy="0 0 0" origin_xyz="-0.135 -0.09 -0.01"
               i_rpy="0 0 0" i_xyz="0 0 0"
-              mass="0.1"
+              mass="0.075"
               c_xyz="0 0 0"
               length="0.044"
@@ -245,5 +245,5 @@
               origin_rpy="0 0 0" origin_xyz="-0.125 -0.15 -0.02"
               i_rpy="0 0 0" i_xyz="0.0 0.0 -0.050"
-              mass="0.05"
+              mass="0.005"
               c_xyz="0.0 0.0 -0.050"
               length="0.028"
@@ -257,5 +257,5 @@
               origin_rpy="0 0 0" origin_xyz="-0.125 -0.15 -0.02"
               i_rpy="0 0 0" i_xyz="0.0 0.0 -0.050"
-              mass="0.15"
+              mass="0.08"
               c_xyz="0.0 0.0 -0.050"
               length="0.028"
@@ -269,5 +269,5 @@
               origin_rpy="0 0 0" origin_xyz="-0.120 -0.15 0.1"
               i_rpy="0 0 0" i_xyz="0.0 0.0 -0.050"
-              mass="0.1"
+              mass="0.034"
               c_xyz="0.0 0.0 -0.050"
               length="0.026"
@@ -281,5 +281,5 @@
               origin_rpy="0 -0.40010 0" origin_xyz="0 -0.01 0"
               i_rpy="0 0 0" i_xyz="0 0 0"
-              mass="0.05"
+              mass="0.0044"
               c_xyz="0 0 0"
               length="0.02"
@@ -305,5 +305,5 @@
   <!-- FRONT LEFT LEG -->
   <!-- SHOULDER TO BASE -->
-  <xacro:rev_joint name="motor_front_left_shoulder" number="0" type="revolute"
+  <xacro:rev_joint name="motor_front_left_shoulder" type="revolute"
                     axis_xyz="1 0 0"
                     origin_rpy="0 0 0" origin_xyz="-0.093 -0.036 0"
@@ -312,8 +312,8 @@
                     damping="0.5"
                     friction="0.5"
-                    lower="-0.548"
-                    upper="0.548"/>
+                    lower="-1.0"
+                    upper="1.0"/>
   <!-- SHOULDER TO LEG -->
-  <xacro:rev_joint name="motor_front_left_leg" number="0" type="revolute"
+  <xacro:rev_joint name="motor_front_left_leg" type="revolute"
                     axis_xyz="0 1 0"
                     origin_rpy="0 0 0" origin_xyz="0 -0.052 0"
@@ -329,5 +329,5 @@
                     parent="front_left_leg_link" child="front_left_leg_link_cover"/>
   <!-- LEG TO FOOT -->
-  <xacro:rev_joint name="foot_motor_front_left" number="0" type="revolute"
+  <xacro:rev_joint name="foot_motor_front_left" type="revolute"
                     axis_xyz="0 1 0"
                     origin_rpy="0 0 0" origin_xyz="-0.01 0 -0.12"
@@ -344,5 +344,5 @@
   <!-- FRONT RIGHT LEG -->
   <!-- SHOULDER TO BASE -->
-  <xacro:rev_joint name="motor_front_right_shoulder" number="0" type="revolute"
+  <xacro:rev_joint name="motor_front_right_shoulder" type="revolute"
                     axis_xyz="1 0 0"
                     origin_rpy="0 0 0" origin_xyz="-0.093 0.036 0"
@@ -351,8 +351,8 @@
                     damping="0.5"
                     friction="0.5"
-                    lower="-0.548"
-                    upper="0.548"/>
+                    lower="-1.0"
+                    upper="1.0"/>
   <!-- SHOULDER TO LEG -->
-  <xacro:rev_joint name="motor_front_right_leg" number="0" type="revolute"
+  <xacro:rev_joint name="motor_front_right_leg" type="revolute"
                     axis_xyz="0 1 0"
                     origin_rpy="0 0 0" origin_xyz="0 0.052 0"
@@ -368,5 +368,5 @@
                     parent="front_right_leg_link" child="front_right_leg_link_cover"/>
   <!-- LEG TO FOOT -->
-  <xacro:rev_joint name="foot_motor_front_right" number="0" type="revolute"
+  <xacro:rev_joint name="foot_motor_front_right" type="revolute"
                     axis_xyz="0 1 0"
                     origin_rpy="0 0 0" origin_xyz="-0.01 0 -0.12"
@@ -383,5 +383,5 @@
   <!-- REAR LEFT LEG -->
   <!-- SHOULDER TO BASE -->
-  <xacro:rev_joint name="motor_rear_left_shoulder" number="0" type="revolute"
+  <xacro:rev_joint name="motor_rear_left_shoulder" type="revolute"
                     axis_xyz="1 0 0"
                     origin_rpy="0 0 0" origin_xyz="0.093 -0.036 0"
@@ -390,8 +390,8 @@
                     damping="0.5"
                     friction="0.5"
-                    lower="-0.548"
-                    upper="0.548"/>
+                    lower="-1.0"
+                    upper="1.0"/>
   <!-- SHOULDER TO LEG -->
-  <xacro:rev_joint name="motor_rear_left_leg" number="0" type="revolute"
+  <xacro:rev_joint name="motor_rear_left_leg" type="revolute"
                     axis_xyz="0 1 0"
                     origin_rpy="0 0 0" origin_xyz="0 -0.052 0"
@@ -407,5 +407,5 @@
                     parent="rear_left_leg_link" child="rear_left_leg_link_cover"/>
   <!-- LEG TO FOOT -->
-  <xacro:rev_joint name="foot_motor_rear_left" number="0" type="revolute"
+  <xacro:rev_joint name="foot_motor_rear_left" type="revolute"
                     axis_xyz="0 1 0"
                     origin_rpy="0 0 0" origin_xyz="-0.01 0 -0.12"
@@ -422,5 +422,5 @@
   <!-- REAR RIGHT LEG -->
   <!-- SHOULDER TO BASE -->
-  <xacro:rev_joint name="motor_rear_right_shoulder" number="0" type="revolute"
+  <xacro:rev_joint name="motor_rear_right_shoulder" type="revolute"
                     axis_xyz="1 0 0"
                     origin_rpy="0 0 0" origin_xyz="0.093 0.036 0"
@@ -429,8 +429,8 @@
                     damping="0.5"
                     friction="0.5"
-                    lower="-0.548"
-                    upper="0.548"/>
+                    lower="-1.0"
+                    upper="1.0"/>
   <!-- SHOULDER TO LEG -->
-  <xacro:rev_joint name="motor_rear_right_leg" number="0" type="revolute"
+  <xacro:rev_joint name="motor_rear_right_leg" type="revolute"
                     axis_xyz="0 1 0"
                     origin_rpy="0 0 0" origin_xyz="0 0.052 0"
@@ -446,5 +446,5 @@
                     parent="rear_right_leg_link" child="rear_right_leg_link_cover"/>
   <!-- LEG TO FOOT -->
-  <xacro:rev_joint name="foot_motor_rear_right" number="0" type="revolute"
+  <xacro:rev_joint name="foot_motor_rear_right" type="revolute"
                     axis_xyz="0 1 0"
                     origin_rpy="0 0 0" origin_xyz="-0.01 0 -0.12"

File: mini_ros/urdf/spot_macro.xacro (robot description, xacro)
@@ -10,5 +10,5 @@
     <color rgba="0.6 0.6 0.6 1"/>
   </material>
-  <xacro:macro name="rev_joint" params="name number type axis_xyz origin_rpy origin_xyz parent child effort velocity damping friction upper lower">
+  <xacro:macro name="rev_joint" params="name type axis_xyz origin_rpy origin_xyz parent child effort velocity damping friction upper lower">
     <joint name="${name}" type="${type}">
       <axis xyz="${axis_xyz}" />
@@ -19,13 +19,4 @@
       <joint_properties damping="${damping}" friction="${friction}" />
     </joint>
-    <transmission name="tran${number}">
-    <type>transmission_interface/SimpleTransmission</type>
-    <joint name="${name}">
-      <hardwareInterface>hardware_interface/EffortJointInterface</hardwareInterface>
-    </joint>
-    <actuator name="motor${number}">
-      <mechanicalReduction>1</mechanicalReduction>
-    </actuator>
-    </transmission>
   </xacro:macro>
   <xacro:macro name="frame_joint" params="name type origin_rpy origin_xyz parent child">
@@ -72,4 +63,5 @@
           <sphere radius="${radius}"/>
         </geometry>
+        <contact_coefficients mu="10.1"/>
       </collision>
       <inertial>
