Commit message: ready for training. Will fork into 'spot' branch for this. Now training on motor model, need to create framework for leg poses

File: bullet/src/spotmicro/util/pybullet_data/assets/urdf/spot.urdf (robot description, URDF)
Before this commit: robot rex, 23 links, 22 joints
Links:
- link base_link: mass 2.80 -> 1.20
- link chassis_front_link: mass 0.20 -> 0.05
- link chassis_rear_link: mass 0.20 -> 0.05
- link front_left_leg_link: mass 0.15 -> 0.1
- link front_left_toe_link: mass 0.05 -> 0.005
- link front_right_leg_link: mass 0.15 -> 0.1
- link front_right_toe_link: mass 0.05 -> 0.005
- link rear_left_leg_link: mass 0.15 -> 0.10
- link rear_left_toe_link: mass 0.05 -> 0.005
- link rear_right_leg_link: mass 0.15 -> 0.10
- link rear_right_toe_link: mass 0.05 -> 0.005

File: mini_ros/urdf/spot.urdf (robot description, URDF)
Before this commit: robot spot, 24 links, 23 joints
Links:
- link base_link: mass 1.2 -> 2.8
- link chassis_front_link: mass 0.05 -> 0.2
- link chassis_rear_link: mass 0.05 -> 0.2
- link front_left_foot_link: mass 0.034 -> 0.1
- link front_left_leg_link: mass 0.08 -> 0.15
- link front_left_shoulder_link: mass 0.075 -> 0.1
- link front_left_toe_link: mass 0.0044 -> 0.05
- link front_right_foot_link: mass 0.034 -> 0.1
- link front_right_leg_link: mass 0.08 -> 0.15
- link front_right_shoulder_link: mass 0.075 -> 0.1
- link front_right_toe_link: mass 0.0044 -> 0.05
- link rear_left_foot_link: mass 0.034 -> 0.1
- link rear_left_leg_link: mass 0.08 -> 0.15
- link rear_left_shoulder_link: mass 0.075 -> 0.1
- link rear_left_toe_link: mass 0.0044 -> 0.05
- link rear_right_foot_link: mass 0.034 -> 0.15
- link rear_right_leg_link: mass 0.08 -> 0.15
- link rear_right_shoulder_link: mass 0.075 -> 0.1
- link rear_right_toe_link: mass 0.0044 -> 0.05
Joints:
- joint foot_motor_front_left: limit lower=-0.1 upper=2.59 effort=1000.0 velocity=0.5 -> lower=-0.1 upper=2.59 effort=1000.0 velocity=0.7
- joint foot_motor_front_right: limit lower=-0.1 upper=2.59 effort=1000.0 velocity=0.5 -> lower=-0.1 upper=2.59 effort=1000.0 velocity=0.7
- joint foot_motor_rear_left: limit lower=-0.1 upper=2.59 effort=1000.0 velocity=0.5 -> lower=-0.1 upper=2.59 effort=1000.0 velocity=0.7
- joint foot_motor_rear_right: limit lower=-0.1 upper=2.59 effort=1000.0 velocity=0.5 -> lower=-0.1 upper=2.59 effort=1000.0 velocity=0.7
- joint motor_front_left_leg: limit lower=-2.17 upper=0.97 effort=3.53 velocity=9.52 -> lower=-2.17 upper=0.97 effort=1000.0 velocity=0.7
- joint motor_front_left_shoulder: limit lower=-1.0 upper=1.0 effort=3.53 velocity=9.52 -> lower=-1.0 upper=1.0 effort=1000.0 velocity=0.7
- joint motor_front_right_leg: limit lower=-2.17 upper=0.97 effort=3.53 velocity=9.52 -> lower=-2.17 upper=0.97 effort=1000.0 velocity=0.7
- joint motor_front_right_shoulder: limit lower=-1.0 upper=1.0 effort=3.53 velocity=9.52 -> lower=-1.0 upper=1.0 effort=1000.0 velocity=0.7
- joint motor_rear_left_leg: limit lower=-2.17 upper=0.97 effort=3.53 velocity=9.52 -> lower=-2.17 upper=0.97 effort=1000.0 velocity=0.7
- joint motor_rear_left_shoulder: limit lower=-1.0 upper=1.0 effort=3.53 velocity=9.52 -> lower=-1.0 upper=1.0 effort=1000.0 velocity=0.7
- joint motor_rear_right_leg: limit lower=-2.17 upper=0.97 effort=3.53 velocity=9.52 -> lower=-2.17 upper=0.97 effort=1000.0 velocity=0.7
- joint motor_rear_right_shoulder: limit lower=-1.0 upper=1.0 effort=3.53 velocity=9.52 -> lower=-1.0 upper=1.0 effort=1000.0 velocity=0.7

File: mini_ros/urdf/spot.urdf.xacro (robot description, xacro)
@@ -10,5 +10,5 @@
               origin_rpy="0 0 0" origin_xyz="-0.045 -0.060 -0.015"
               i_rpy="0 0 0" i_xyz="0 0 0"
-              mass="1.2"
+              mass="2.8"
               c_xyz="0 0 0"
               length="0.14"
@@ -22,5 +22,5 @@
               origin_rpy="0 0 0" origin_xyz="-0.040 -0.060 -0.0140"
               i_rpy="0 0 0" i_xyz="-0.145 0 0"
-              mass="0.05"
+              mass="0.2"
               c_xyz="-0.145 0 0"
               length="0.058"
@@ -34,5 +34,5 @@
               origin_rpy="0 0 0" origin_xyz="-0.040 -0.060 -0.0140"
               i_rpy="0 0 0" i_xyz="0.135 0 0"
-              mass="0.05"
+              mass="0.2"
               c_xyz="0.135 0 0"
               length="0.04"
@@ -47,5 +47,5 @@
               origin_rpy="0 0 0" origin_xyz="-0.135 -0.02 -0.01"
               i_rpy="0 0 0" i_xyz="0 0 0"
-              mass="0.075"
+              mass="0.1"
               c_xyz="0 0 0"
               length="0.044"
@@ -71,5 +71,5 @@
               origin_rpy="0 0 0" origin_xyz="-0.125 0.04 -0.02"
               i_rpy="0 0 0" i_xyz="0.0 0.0 -0.050"
-              mass="0.08"
+              mass="0.15"
               c_xyz="0.0 0.0 -0.050"
               length="0.028"
@@ -83,5 +83,5 @@
               origin_rpy="0 0 0" origin_xyz="-0.120 0.04 0.1"
               i_rpy="0 0 0" i_xyz="0.0 0.0 -0.050"
-              mass="0.034"
+              mass="0.1"
               c_xyz="0.0 0.0 -0.050"
               length="0.026"
@@ -95,5 +95,5 @@
               origin_rpy="0 -0.40010 0" origin_xyz="0 -0.01 0"
               i_rpy="0 0 0" i_xyz="0 0 0"
-              mass="0.0044"
+              mass="0.05"
               c_xyz="0 0 0"
               length="0.02"
@@ -109,5 +109,5 @@
               origin_rpy="0 0 0" origin_xyz="-0.135 -0.09 -0.01"
               i_rpy="0 0 0" i_xyz="0 0 0"
-              mass="0.075"
+              mass="0.1"
               c_xyz="0 0 0"
               length="0.044"
@@ -133,5 +133,5 @@
               origin_rpy="0 0 0" origin_xyz="-0.125 -0.15 -0.02"
               i_rpy="0 0 0" i_xyz="0.0 0.0 -0.050"
-              mass="0.08"
+              mass="0.15"
               c_xyz="0.0 0.0 -0.050"
               length="0.028"
@@ -145,5 +145,5 @@
               origin_rpy="0 0 0" origin_xyz="-0.120 -0.15 0.1"
               i_rpy="0 0 0" i_xyz="0.0 0.0 -0.050"
-              mass="0.034"
+              mass="0.1"
               c_xyz="0.0 0.0 -0.050"
               length="0.026"
@@ -157,5 +157,5 @@
               origin_rpy="0 -0.40010 0" origin_xyz="0 -0.01 0"
               i_rpy="0 0 0" i_xyz="0 0 0"
-              mass="0.0044"
+              mass="0.05"
               c_xyz="0 0 0"
               length="0.02"
@@ -171,5 +171,5 @@
               origin_rpy="0 0 0" origin_xyz="-0.135 -0.02 -0.01"
               i_rpy="0 0 0" i_xyz="0 0 0"
-              mass="0.075"
+              mass="0.1"
               c_xyz="0 0 0"
               length="0.044"
@@ -195,5 +195,5 @@
               origin_rpy="0 0 0" origin_xyz="-0.125 0.04 -0.02"
               i_rpy="0 0 0" i_xyz="0.0 0.0 -0.050"
-              mass="0.08"
+              mass="0.15"
               c_xyz="0.0 0.0 -0.050"
               length="0.028"
@@ -207,5 +207,5 @@
               origin_rpy="0 0 0" origin_xyz="-0.120 0.04 0.1"
               i_rpy="0 0 0" i_xyz="0.0 0.0 -0.050"
-              mass="0.034"
+              mass="0.1"
               c_xyz="0.0 0.0 -0.050"
               length="0.026"
@@ -219,5 +219,5 @@
               origin_rpy="0 -0.40010 0" origin_xyz="0 -0.01 0"
               i_rpy="0 0 0" i_xyz="0 0 0"
-              mass="0.0044"
+              mass="0.05"
               c_xyz="0 0 0"
               length="0.02"
@@ -233,5 +233,5 @@
               origin_rpy="0 0 0" origin_xyz="-0.135 -0.09 -0.01"
               i_rpy="0 0 0" i_xyz="0 0 0"
-              mass="0.075"
+              mass="0.1"
               c_xyz="0 0 0"
               length="0.044"
@@ -257,5 +257,5 @@
               origin_rpy="0 0 0" origin_xyz="-0.125 -0.15 -0.02"
               i_rpy="0 0 0" i_xyz="0.0 0.0 -0.050"
-              mass="0.08"
+              mass="0.15"
               c_xyz="0.0 0.0 -0.050"
               length="0.028"
@@ -269,5 +269,5 @@
               origin_rpy="0 0 0" origin_xyz="-0.120 -0.15 0.1"
               i_rpy="0 0 0" i_xyz="0.0 0.0 -0.050"
-              mass="0.034"
+              mass="0.15"
               c_xyz="0.0 0.0 -0.050"
               length="0.026"
@@ -281,5 +281,5 @@
               origin_rpy="0 -0.40010 0" origin_xyz="0 -0.01 0"
               i_rpy="0 0 0" i_xyz="0 0 0"
-              mass="0.0044"
+              mass="0.05"
               c_xyz="0 0 0"
               length="0.02"
@@ -309,7 +309,7 @@
                     origin_rpy="0 0 0" origin_xyz="-0.093 -0.036 0"
                     parent="base_link" child="front_left_shoulder_link"
-                    effort="3.530" velocity="9.52"
-                    damping="0.5"
-                    friction="0.5"
+                    effort="1000.0" velocity="0.7"
+                    damping="0.0"
+                    friction="0.0"
                     lower="-1.0"
                     upper="1.0"/>
@@ -319,7 +319,7 @@
                     origin_rpy="0 0 0" origin_xyz="0 -0.052 0"
                     parent="front_left_shoulder_link" child="front_left_leg_link"
-                    effort="3.530" velocity="9.52"
-                    damping="0.5"
-                    friction="0.5"
+                    effort="1000.0" velocity="0.7"
+                    damping="0.0"
+                    friction="0.0"
                     lower="-2.17"
                     upper="0.97"/>
@@ -333,7 +333,7 @@
                     origin_rpy="0 0 0" origin_xyz="-0.01 0 -0.12"
                     parent="front_left_leg_link" child="front_left_foot_link"
-                    effort="3.530" velocity="9.52"
-                    damping="0.5"
-                    friction="0.5"
+                    effort="1000.0" velocity="0.7"
+                    damping="0.0"
+                    friction="0.0"
                     lower="-0.1"
                     upper="2.59"/>
@@ -348,7 +348,7 @@
                     origin_rpy="0 0 0" origin_xyz="-0.093 0.036 0"
                     parent="base_link" child="front_right_shoulder_link"
-                    effort="3.530" velocity="9.52"
-                    damping="0.5"
-                    friction="0.5"
+                    effort="1000.0" velocity="0.7"
+                    damping="0.0"
+                    friction="0.0"
                     lower="-1.0"
                     upper="1.0"/>
@@ -358,7 +358,7 @@
                     origin_rpy="0 0 0" origin_xyz="0 0.052 0"
                     parent="front_right_shoulder_link" child="front_right_leg_link"
-                    effort="3.530" velocity="9.52"
-                    damping="0.5"
-                    friction="0.5"
+                    effort="1000.0" velocity="0.7"
+                    damping="0.0"
+                    friction="0.0"
                     lower="-2.17"
                     upper="0.97"/>
@@ -372,7 +372,7 @@
                     origin_rpy="0 0 0" origin_xyz="-0.01 0 -0.12"
                     parent="front_right_leg_link" child="front_right_foot_link"
-                    effort="3.530" velocity="9.52"
-                    damping="0.5"
-                    friction="0.5"
+                    effort="1000.0" velocity="0.7"
+                    damping="0.0"
+                    friction="0.0"
                     lower="-0.1"
                     upper="2.59"/>
@@ -387,7 +387,7 @@
                     origin_rpy="0 0 0" origin_xyz="0.093 -0.036 0"
                     parent="base_link" child="rear_left_shoulder_link"
-                    effort="3.530" velocity="9.52"
-                    damping="0.5"
-                    friction="0.5"
+                    effort="1000.0" velocity="0.7"
+                    damping="0.0"
+                    friction="0.0"
                     lower="-1.0"
                     upper="1.0"/>
@@ -397,7 +397,7 @@
                     origin_rpy="0 0 0" origin_xyz="0 -0.052 0"
                     parent="rear_left_shoulder_link" child="rear_left_leg_link"
-                    effort="3.530" velocity="9.52"
-                    damping="0.5"
-                    friction="0.5"
+                    effort="1000.0" velocity="0.7"
+                    damping="0.0"
+                    friction="0.0"
                     lower="-2.17"
                     upper="0.97"/>
@@ -411,7 +411,7 @@
                     origin_rpy="0 0 0" origin_xyz="-0.01 0 -0.12"
                     parent="rear_left_leg_link" child="rear_left_foot_link"
-                    effort="3.530" velocity="9.52"
-                    damping="0.5"
-                    friction="0.5"
+                    effort="1000.0" velocity="0.7"
+                    damping="0.0"
+                    friction="0.0"
                     lower="-0.1"
                     upper="2.59"/>
@@ -426,7 +426,7 @@
                     origin_rpy="0 0 0" origin_xyz="0.093 0.036 0"
                     parent="base_link" child="rear_right_shoulder_link"
-                    effort="3.530" velocity="9.52"
-                    damping="0.5"
-                    friction="0.5"
+                    effort="1000.0" velocity="0.7"
+                    damping="0.0"
+                    friction="0.0"
                     lower="-1.0"
                     upper="1.0"/>
@@ -436,7 +436,7 @@
                     origin_rpy="0 0 0" origin_xyz="0 0.052 0"
                     parent="rear_right_shoulder_link" child="rear_right_leg_link"
-                    effort="3.530" velocity="9.52"
-                    damping="0.5"
-                    friction="0.5"
+                    effort="1000.0" velocity="0.7"
+                    damping="0.0"
+                    friction="0.0"
                     lower="-2.17"
                     upper="0.97"/>
@@ -450,7 +450,7 @@
                     origin_rpy="0 0 0" origin_xyz="-0.01 0 -0.12"
                     parent="rear_right_leg_link" child="rear_right_foot_link"
-                    effort="3.530" velocity="9.52"
-                    damping="0.5"
-                    friction="0.5"
+                    effort="1000.0" velocity="0.7"
+                    damping="0.0"
+                    friction="0.0"
                     lower="-0.1"
                     upper="2.59"/>

File: mini_ros/urdf/spot_macro.xacro (robot description, xacro)
@@ -45,5 +45,5 @@
         <mass value="${mass}" />
         <origin rpy="${i_rpy}" xyz="${i_xyz}" /> <!-- Inertial Axes -->
-        <inertia ixx="${mass * (length * length + height * height)/12}" ixy="${0}" ixz="${0}" iyx="${0}" iyy="${mass * (length * length + height * height)/12}" iyz="${0}" izx="${0}" izy="${0}" izz="${mass * (length * length + width * width)/12}" />
+        <inertia ixx="${mass * (width * width + height * height)/12.0}" ixy="${0}" ixz="${0}" iyx="${0}" iyy="${mass * (length * length + height * height)/12.0}" iyz="${0}" izx="${0}" izy="${0}" izz="${mass * (length * length + width * width)/12.0}" />
       </inertial>
     </link>
@@ -68,5 +68,5 @@
         <mass value="${mass}" />
         <origin rpy="${i_rpy}" xyz="${i_xyz}" /> <!-- Inertial Axes -->
-        <inertia ixx="${mass * (length * length + height * height)/12}" ixy="${0}" ixz="${0}" iyx="${0}" iyy="${mass * (length * length + height * height)/12}" iyz="${0}" izx="${0}" izy="${0}" izz="${mass * (length * length + width * width)/12}" />
+        <inertia ixx="${mass * (width * width + height * height)/12.0}" ixy="${0}" ixz="${0}" iyx="${0}" iyy="${mass * (length * length + height * height)/12.0}" iyz="${0}" izx="${0}" izy="${0}" izz="${mass * (length * length + width * width)/12.0}" />
       </inertial>
     </link>

Commit message: added testing and training scripts using ARS for spot. also added joint limit enforcer in gym env

File: bullet/src/spotmicro/util/pybullet_data/assets/urdf/spot.urdf (robot description, URDF)
Before this commit: robot rex, 23 links, 22 joints
Joints:
- joint motor_front_left_leg: limit lower=-2.666 upper=1.548 effort=1000.0 velocity=0.5 -> lower=-2.17 upper=0.97 effort=1000.0 velocity=0.5
- joint motor_front_left_shoulder: limit lower=-0.548 upper=0.548 effort=1000.0 velocity=0.7 -> lower=-1.0 upper=1.0 effort=1000.0 velocity=0.7
- joint motor_front_right_leg: limit lower=-2.666 upper=1.548 effort=1000.0 velocity=0.5 -> lower=-2.17 upper=0.97 effort=1000.0 velocity=0.5
- joint motor_front_right_shoulder: limit lower=-0.548 upper=0.548 effort=1000.0 velocity=0.7 -> lower=-1.0 upper=1.0 effort=1000.0 velocity=0.7
- joint motor_rear_left_leg: limit lower=-2.666 upper=1.548 effort=1000.0 velocity=0.5 -> lower=-2.17 upper=0.97 effort=1000.0 velocity=0.5
- joint motor_rear_left_shoulder: limit lower=-0.548 upper=0.548 effort=1000.0 velocity=0.7 -> lower=-1.0 upper=1.0 effort=1000.0 velocity=0.7
- joint motor_rear_right_leg: limit lower=-2.666 upper=1.548 effort=1000.0 velocity=0.5 -> lower=-2.17 upper=0.97 effort=1000.0 velocity=0.5
- joint motor_rear_right_shoulder: limit lower=-0.548 upper=0.548 effort=1000.0 velocity=0.7 -> lower=-1.0 upper=1.0 effort=1000.0 velocity=0.7

Commit message: draft 1 of Bezier Gait. Issue with calculating TD event time

File: bullet/src/spotmicro/util/pybullet_data/assets/urdf/spot.urdf (robot description, URDF)
Before this commit: robot rex, 23 links, 22 joints
Links:
- link front_left_toe_link: geometry collision mesh filename=stl/foot.stl scale=0.001 0.001 0.001; visual mesh filename=stl/foot.stl scale=0.001 0.001 0.001
- link front_right_toe_link: geometry collision mesh filename=stl/foot.stl scale=0.001 0.001 0.001; visual mesh filename=stl/foot.stl scale=0.001 0.001 0.001
- link rear_left_toe_link: geometry collision mesh filename=stl/foot.stl scale=0.001 0.001 0.001; visual mesh filename=stl/foot.stl scale=0.001 0.001 0.001
- link rear_right_toe_link: geometry collision mesh filename=stl/foot.stl scale=0.001 0.001 0.001; visual mesh filename=stl/foot.stl scale=0.001 0.001 0.001

File: mini_ros/urdf/spot.urdf (robot description, URDF)
Before this commit: robot spot, 24 links, 23 joints
Links:
- link base_link: mass 2.8 -> 1.2
- link chassis_front_link: mass 0.2 -> 0.1
- link chassis_rear_link: mass 0.2 -> 0.1
- link front_left_leg_link: mass 0.15 -> 0.1
- link front_left_toe_link: mass 0.05 -> 0.005
- link front_right_leg_link: mass 0.15 -> 0.1
- link front_right_toe_link: mass 0.05 -> 0.005
- link rear_left_leg_link: mass 0.15 -> 0.1
- link rear_left_toe_link: mass 0.05 -> 0.005
- link rear_right_leg_link: mass 0.15 -> 0.1
- link rear_right_toe_link: mass 0.05 -> 0.005
Joints:
- joint foot_motor_front_left: limit lower=-0.1 upper=2.59 effort=1000.0 velocity=0.7 -> lower=-0.1 upper=2.59 effort=3.5 velocity=9.5
- joint foot_motor_front_right: limit lower=-0.1 upper=2.59 effort=1000.0 velocity=0.7 -> lower=-0.1 upper=2.59 effort=3.5 velocity=9.5
- joint foot_motor_rear_left: limit lower=-0.1 upper=2.59 effort=1000.0 velocity=0.7 -> lower=-0.1 upper=2.59 effort=3.5 velocity=9.5
- joint foot_motor_rear_right: limit lower=-0.1 upper=2.59 effort=1000.0 velocity=0.7 -> lower=-0.1 upper=2.59 effort=3.5 velocity=9.5
- joint motor_front_left_leg: limit lower=-2.17 upper=0.97 effort=1000.0 velocity=0.7 -> lower=-2.17 upper=0.97 effort=3.5 velocity=9.5
- joint motor_front_left_shoulder: limit lower=-1.0 upper=1.0 effort=1000.0 velocity=0.7 -> lower=-1.0 upper=1.0 effort=3.5 velocity=9.5
- joint motor_front_right_leg: limit lower=-2.17 upper=0.97 effort=1000.0 velocity=0.7 -> lower=-2.17 upper=0.97 effort=3.5 velocity=9.5
- joint motor_front_right_shoulder: limit lower=-1.0 upper=1.0 effort=1000.0 velocity=0.7 -> lower=-1.0 upper=1.0 effort=3.5 velocity=9.5
- joint motor_rear_left_leg: limit lower=-2.17 upper=0.97 effort=1000.0 velocity=0.7 -> lower=-2.17 upper=0.97 effort=3.5 velocity=9.5
- joint motor_rear_left_shoulder: limit lower=-1.0 upper=1.0 effort=1000.0 velocity=0.7 -> lower=-1.0 upper=1.0 effort=3.5 velocity=9.5
- joint motor_rear_right_leg: limit lower=-2.17 upper=0.97 effort=1000.0 velocity=0.7 -> lower=-2.17 upper=0.97 effort=3.5 velocity=9.5
- joint motor_rear_right_shoulder: limit lower=-1.0 upper=1.0 effort=1000.0 velocity=0.7 -> lower=-1.0 upper=1.0 effort=3.5 velocity=9.5

File: mini_ros/urdf/spot.urdf.xacro (robot description, xacro)
@@ -10,5 +10,5 @@
               origin_rpy="0 0 0" origin_xyz="-0.045 -0.060 -0.015"
               i_rpy="0 0 0" i_xyz="0 0 0"
-              mass="2.8"
+              mass="1.2"
               c_xyz="0 0 0"
               length="0.14"
@@ -22,5 +22,5 @@
               origin_rpy="0 0 0" origin_xyz="-0.040 -0.060 -0.0140"
               i_rpy="0 0 0" i_xyz="-0.145 0 0"
-              mass="0.2"
+              mass="0.1"
               c_xyz="-0.145 0 0"
               length="0.058"
@@ -34,5 +34,5 @@
               origin_rpy="0 0 0" origin_xyz="-0.040 -0.060 -0.0140"
               i_rpy="0 0 0" i_xyz="0.135 0 0"
-              mass="0.2"
+              mass="0.1"
               c_xyz="0.135 0 0"
               length="0.04"
@@ -71,5 +71,5 @@
               origin_rpy="0 0 0" origin_xyz="-0.125 0.04 -0.02"
               i_rpy="0 0 0" i_xyz="0.0 0.0 -0.050"
-              mass="0.15"
+              mass="0.1"
               c_xyz="0.0 0.0 -0.050"
               length="0.028"
@@ -95,5 +95,5 @@
               origin_rpy="0 -0.40010 0" origin_xyz="0 -0.01 0"
               i_rpy="0 0 0" i_xyz="0 0 0"
-              mass="0.05"
+              mass="0.005"
               c_xyz="0 0 0"
               length="0.02"
@@ -133,5 +133,5 @@
               origin_rpy="0 0 0" origin_xyz="-0.125 -0.15 -0.02"
               i_rpy="0 0 0" i_xyz="0.0 0.0 -0.050"
-              mass="0.15"
+              mass="0.1"
               c_xyz="0.0 0.0 -0.050"
               length="0.028"
@@ -157,5 +157,5 @@
               origin_rpy="0 -0.40010 0" origin_xyz="0 -0.01 0"
               i_rpy="0 0 0" i_xyz="0 0 0"
-              mass="0.05"
+              mass="0.005"
               c_xyz="0 0 0"
               length="0.02"
@@ -195,5 +195,5 @@
               origin_rpy="0 0 0" origin_xyz="-0.125 0.04 -0.02"
               i_rpy="0 0 0" i_xyz="0.0 0.0 -0.050"
-              mass="0.15"
+              mass="0.1"
               c_xyz="0.0 0.0 -0.050"
               length="0.028"
@@ -219,5 +219,5 @@
               origin_rpy="0 -0.40010 0" origin_xyz="0 -0.01 0"
               i_rpy="0 0 0" i_xyz="0 0 0"
-              mass="0.05"
+              mass="0.005"
               c_xyz="0 0 0"
               length="0.02"
@@ -257,5 +257,5 @@
               origin_rpy="0 0 0" origin_xyz="-0.125 -0.15 -0.02"
               i_rpy="0 0 0" i_xyz="0.0 0.0 -0.050"
-              mass="0.15"
+              mass="0.1"
               c_xyz="0.0 0.0 -0.050"
               length="0.028"
@@ -281,5 +281,5 @@
               origin_rpy="0 -0.40010 0" origin_xyz="0 -0.01 0"
               i_rpy="0 0 0" i_xyz="0 0 0"
-              mass="0.05"
+              mass="0.005"
               c_xyz="0 0 0"
               length="0.02"
