Commit message: trained policy to keep straight line (ARS policy # 319) as stock gait drifts left

File: bullet/src/spotmicro/util/pybullet_data/assets/urdf/spot.urdf (robot description, URDF)
Before this commit: robot rex, 23 links, 22 joints
Joints:
- joint foot_motor_front_left: limit lower=-0.1 upper=2.59 effort=1000.0 velocity=0.5 -> lower=-0.1 upper=2.59 effort=100.0 velocity=0.5
- joint foot_motor_front_right: limit lower=-0.1 upper=2.59 effort=1000.0 velocity=0.5 -> lower=-0.1 upper=2.59 effort=100.0 velocity=0.5
- joint foot_motor_rear_left: limit lower=-0.1 upper=2.59 effort=1000.0 velocity=0.5 -> lower=-0.1 upper=2.59 effort=100.0 velocity=0.5
- joint foot_motor_rear_right: limit lower=-0.1 upper=2.59 effort=1000.0 velocity=0.5 -> lower=-0.1 upper=2.59 effort=100.0 velocity=0.5
- joint motor_front_left_leg: limit lower=-2.17 upper=0.97 effort=1000.0 velocity=0.5 -> lower=-2.17 upper=0.97 effort=100.0 velocity=0.5
- joint motor_front_left_shoulder: limit lower=-1.0 upper=1.0 effort=1000.0 velocity=0.7 -> lower=-1.0 upper=1.0 effort=100.0 velocity=0.7
- joint motor_front_right_leg: limit lower=-2.17 upper=0.97 effort=1000.0 velocity=0.5 -> lower=-2.17 upper=0.97 effort=100.0 velocity=0.5
- joint motor_front_right_shoulder: limit lower=-1.0 upper=1.0 effort=1000.0 velocity=0.7 -> lower=-1.0 upper=1.0 effort=100.0 velocity=0.7
- joint motor_rear_left_leg: limit lower=-2.17 upper=0.97 effort=1000.0 velocity=0.5 -> lower=-2.17 upper=0.97 effort=100.0 velocity=0.5
- joint motor_rear_left_shoulder: limit lower=-1.0 upper=1.0 effort=1000.0 velocity=0.7 -> lower=-1.0 upper=1.0 effort=100.0 velocity=0.7
- joint motor_rear_right_leg: limit lower=-2.17 upper=0.97 effort=1000.0 velocity=0.5 -> lower=-2.17 upper=0.97 effort=100.0 velocity=0.5
- joint motor_rear_right_shoulder: limit lower=-1.0 upper=1.0 effort=1000.0 velocity=0.7 -> lower=-1.0 upper=1.0 effort=100.0 velocity=0.7
