Commit message: using original inertial values

File: spotmicro/util/pybullet_data/assets/urdf/spot.urdf (robot description, URDF)
Before this commit: robot spot, 24 links, 23 joints
Links:
- link back: mass 0.025 -> 0.1
- link back_bracket: mass 0.025 -> 0.1
- link back_left_hip: mass 0.120 -> 0.2
- link back_left_lower_leg: mass 0.1 -> 0.05
- link back_left_upper_leg: mass None -> 0.13
- link back_right_hip: mass 0.120 -> 0.2
- link back_right_lower_leg: mass 0.1 -> 0.05
- link back_right_upper_leg: mass None -> 0.13
- link base_link: mass 1.20 -> 0.6
- link chassis_left: mass 0.0001 -> 0.01
- link chassis_right: mass 0.0001 -> 0.01
- link front: mass 0.025 -> 0.1
- link front_bracket: mass 0.025 -> 0.1
- link front_left_hip: mass 0.12 -> 0.2
- link front_left_lower_leg: mass 0.1 -> 0.05
- link front_left_upper_leg: mass None -> 0.13
- link front_right_hip: mass 0.120 -> 0.2
- link front_right_lower_leg: mass 0.1 -> 0.05
- link front_right_upper_leg: mass None -> 0.13
