Commit message: fixed bugs, good walking performance. invisible STL problem still present

File: mini_ros/urdf/spot_macro.xacro (robot description, xacro)
@@ -61,5 +61,5 @@
         <origin rpy="${origin_rpy}" xyz="${c_xyz}" />
         <geometry>
-          <sphere radius="${radius}"/>
+          <mesh filename="${meshfile}" scale="${meshscale}"/>
         </geometry>
         <contact_coefficients mu="10.1"/>

File: spotmicro/util/pybullet_data/assets/urdf/spot.urdf (robot description, URDF)
Before this commit: robot spot, 24 links, 23 joints
Links:
- link back: mass 0.1 -> 0.025; geometry collision box size=0.114 0.075 0.085; visual mesh filename=stl/OpenQuadruped/Back.stl scale=1 1 1
- link back_bracket: mass 0.1 -> 0.025; geometry collision box size=0.025 0.075 0.085; visual mesh filename=stl/OpenQuadruped/Back_Bracket.stl scale=1 1 1
- link back_left_foot: geometry collision mesh filename=stl/OpenQuadruped/LEFT_FOOT.stl scale=1 1 1; visual mesh filename=stl/OpenQuadruped/LEFT_FOOT.stl scale=1 1 1
- link back_left_hip: mass 0.2 -> 0.120; geometry collision box size=0.05 0.065 0.065; visual mesh filename=stl/OpenQuadruped/LEFT_HIP.stl scale=1 1 1
- link back_left_lower_leg: mass 0.05 -> 0.1; geometry collision box size=0.035 0.035 0.12; visual mesh filename=stl/OpenQuadruped/LEFT_LOWER_LEG.stl scale=1 1 1
- link back_left_upper_leg: mass 0.13 -> None; geometry collision box size=0.035 0.035 0.11; visual mesh filename=stl/OpenQuadruped/LEFT_UPPER_LEG.stl scale=1 1 1
- link back_right_foot: geometry collision mesh filename=stl/OpenQuadruped/RIGHT_FOOT.stl scale=1 1 1; visual mesh filename=stl/OpenQuadruped/RIGHT_FOOT.stl scale=1 1 1
- link back_right_hip: mass 0.2 -> 0.120; geometry collision box size=0.05 0.065 0.065; visual mesh filename=stl/OpenQuadruped/RIGHT_HIP.stl scale=1 1 1
- link back_right_lower_leg: mass 0.05 -> 0.1; geometry collision box size=0.035 0.035 0.12; visual mesh filename=stl/OpenQuadruped/RIGHT_LOWER_LEG.stl scale=1 1 1
- link back_right_upper_leg: mass 0.13 -> None; geometry collision box size=0.035 0.035 0.11; visual mesh filename=stl/OpenQuadruped/RIGHT_UPPER_LEG.stl scale=1 1 1
- link base_link: mass 0.6 -> 1.20; geometry collision box size=0.114 0.2 0.1; visual mesh filename=stl/OpenQuadruped/MAINBODY.stl scale=1 1 1
- link battery: geometry collision box size=0.048 0.145 0.026; visual mesh filename=stl/OpenQuadruped/Battery.stl scale=1 1 1
- link chassis_left: mass 0.01 -> 0.0001; geometry collision box size=0.06 0.15 0.006; visual mesh filename=stl/OpenQuadruped/Chassis_Left_Side.stl scale=1 1 1
- link chassis_right: mass 0.01 -> 0.0001; geometry collision box size=0.06 0.15 0.006; visual mesh filename=stl/OpenQuadruped/Chassis_Right_Side.stl scale=1 1 1
- link front: mass 0.1 -> 0.025; geometry collision box size=0.114 0.045 0.085; visual mesh filename=stl/OpenQuadruped/Front.stl scale=1 1 1
- link front_bracket: mass 0.1 -> 0.025; geometry collision box size=0.025 0.075 0.085; visual mesh filename=stl/OpenQuadruped/Front_Bracket.stl scale=1 1 1
- link front_left_foot: geometry collision mesh filename=stl/OpenQuadruped/LEFT_FOOT.stl scale=1 1 1; visual mesh filename=stl/OpenQuadruped/LEFT_FOOT.stl scale=1 1 1
- link front_left_hip: mass 0.2 -> 0.12; geometry collision box size=0.05 0.065 0.065; visual mesh filename=stl/OpenQuadruped/LEFT_HIP.stl scale=1 1 1
- link front_left_lower_leg: mass 0.05 -> 0.1; geometry collision box size=0.035 0.035 0.12; visual mesh filename=stl/OpenQuadruped/LEFT_LOWER_LEG.stl scale=1 1 1
- link front_left_upper_leg: mass 0.13 -> None; geometry collision box size=0.035 0.035 0.11; visual mesh filename=stl/OpenQuadruped/LEFT_UPPER_LEG.stl scale=1 1 1
- link front_right_foot: geometry collision mesh filename=stl/OpenQuadruped/RIGHT_FOOT.stl scale=1 1 1; visual mesh filename=stl/OpenQuadruped/RIGHT_FOOT.stl scale=1 1 1
- link front_right_hip: mass 0.2 -> 0.120; geometry collision box size=0.05 0.065 0.065; visual mesh filename=stl/OpenQuadruped/RIGHT_HIP.stl scale=1 1 1
- link front_right_lower_leg: mass 0.05 -> 0.1; geometry collision box size=0.035 0.035 0.12; visual mesh filename=stl/OpenQuadruped/RIGHT_LOWER_LEG.stl scale=1 1 1
- link front_right_upper_leg: mass 0.13 -> None; geometry collision box size=0.035 0.035 0.11; visual mesh filename=stl/OpenQuadruped/RIGHT_UPPER_LEG.stl scale=1 1 1

Commit message: add explicit declaration of Gazebo color based on matname param

File: mini_ros/urdf/spot_macro.xacro (robot description, xacro)
@@ -48,4 +48,12 @@
       </inertial>
     </link>
+    <gazebo reference="${name}">
+        <xacro:if value="${matname == 'black'}">
+          <material>Gazebo/Black</material>
+        </xacro:if>
+        <xacro:if value="${matname == 'orange'}">
+          <material>Gazebo/Orange</material>
+        </xacro:if>
+    </gazebo>
   </xacro:macro>
   <xacro:macro name="mesh_link_sphere" params="name origin_xyz origin_rpy meshfile meshscale c_xyz matname mass i_xyz i_rpy length width height radius">
