Commit message: fixed joint limits and added spheres as toes

File: mini_ros/urdf/spot.urdf.xacro (robot description, xacro)
@@ -92,5 +92,5 @@
               meshscale="0.001 0.001 0.001" />
 <!-- TOE -->
-  <xacro:mesh_link name="front_left_toe_link"
+  <xacro:mesh_link_sphere name="front_left_toe_link"
               origin_rpy="0 -0.40010 0" origin_xyz="0 -0.01 0"
               i_rpy="0 0 0" i_xyz="0 0 0"
@@ -100,4 +100,5 @@
               width="0.02"
               height="0.02"
+              radius="0.02"
               matname="grey"
               meshfile="package://mini_ros/stl/foot.stl"
@@ -153,5 +154,5 @@
               meshscale="0.001 0.001 0.001" />
 <!-- TOE -->
-  <xacro:mesh_link name="front_right_toe_link"
+  <xacro:mesh_link_sphere name="front_right_toe_link"
               origin_rpy="0 -0.40010 0" origin_xyz="0 -0.01 0"
               i_rpy="0 0 0" i_xyz="0 0 0"
@@ -161,4 +162,5 @@
               width="0.02"
               height="0.02"
+              radius="0.02"
               matname="grey"
               meshfile="package://mini_ros/stl/foot.stl"
@@ -214,5 +216,5 @@
               meshscale="0.001 0.001 0.001" />
 <!-- TOE -->
-  <xacro:mesh_link name="rear_left_toe_link"
+  <xacro:mesh_link_sphere name="rear_left_toe_link"
               origin_rpy="0 -0.40010 0" origin_xyz="0 -0.01 0"
               i_rpy="0 0 0" i_xyz="0 0 0"
@@ -222,4 +224,5 @@
               width="0.02"
               height="0.02"
+              radius="0.02"
               matname="grey"
               meshfile="package://mini_ros/stl/foot.stl"
@@ -275,5 +278,5 @@
               meshscale="0.001 0.001 0.001" />
 <!-- TOE -->
-  <xacro:mesh_link name="rear_right_toe_link"
+  <xacro:mesh_link_sphere name="rear_right_toe_link"
               origin_rpy="0 -0.40010 0" origin_xyz="0 -0.01 0"
               i_rpy="0 0 0" i_xyz="0 0 0"
@@ -283,4 +286,5 @@
               width="0.02"
               height="0.02"
+              radius="0.02"
               matname="grey"
               meshfile="package://mini_ros/stl/foot.stl"
@@ -318,6 +322,6 @@
                     damping="0.5"
                     friction="0.5"
-                    lower="-2.666"
-                    upper="1.548"/>
+                    lower="-2.17"
+                    upper="0.97"/>
   <!-- LEG TO COVER -->
   <xacro:frame_joint name="front_left_leg_cover_joint" type="fixed"
@@ -357,6 +361,6 @@
                     damping="0.5"
                     friction="0.5"
-                    lower="-2.666"
-                    upper="1.548"/>
+                    lower="-2.17"
+                    upper="0.97"/>
   <!-- LEG TO COVER -->
   <xacro:frame_joint name="front_right_leg_cover_joint" type="fixed"
@@ -396,6 +400,6 @@
                     damping="0.5"
                     friction="0.5"
-                    lower="-2.666"
-                    upper="1.548"/>
+                    lower="-2.17"
+                    upper="0.97"/>
   <!-- LEG TO COVER -->
   <xacro:frame_joint name="rear_left_leg_cover_joint" type="fixed"
@@ -435,6 +439,6 @@
                     damping="0.5"
                     friction="0.5"
-                    lower="-2.666"
-                    upper="1.548"/>
+                    lower="-2.17"
+                    upper="0.97"/>
   <!-- LEG TO COVER -->
   <xacro:frame_joint name="rear_right_leg_cover_joint" type="fixed"

File: mini_ros/urdf/spot_macro.xacro (robot description, xacro)
@@ -58,3 +58,25 @@
     </link>
   </xacro:macro>
+  <xacro:macro name="mesh_link_sphere" params="name origin_xyz origin_rpy meshfile meshscale c_xyz matname mass i_xyz i_rpy length width height radius">
+    <link name="${name}">
+      <visual>
+        <origin rpy="${origin_rpy}" xyz="${origin_xyz}" />
+        <geometry>
+          <mesh filename="${meshfile}" scale="${meshscale}"/>
+        </geometry>
+        <material name="${matname}"/>
+      </visual>
+      <collision>
+        <origin rpy="${origin_rpy}" xyz="${c_xyz}" />
+        <geometry>
+          <sphere radius="${radius}"/>
+        </geometry>
+      </collision>
+      <inertial>
+        <mass value="${mass}" />
+        <origin rpy="${i_rpy}" xyz="${i_xyz}" /> <!-- Inertial Axes -->
+        <inertia ixx="${mass * (length * length + height * height)/12}" ixy="${0}" ixz="${0}" iyx="${0}" iyy="${mass * (length * length + height * height)/12}" iyz="${0}" izx="${0}" izy="${0}" izz="${mass * (length * length + width * width)/12}" />
+      </inertial>
+    </link>
+  </xacro:macro>
 </robot>

Commit message: removed inertia from root link and shifted to new base_inertia link

File: mini_ros/urdf/spot.urdf.xacro (robot description, xacro)
@@ -5,7 +5,7 @@
   <!-- Robot description -->
   <!-- STATIC Links -->
-  <link name="base_footprint"/>
+  <link name="base_link"/>
   <!-- MAIN BODY -->
-  <xacro:mesh_link name="base_link"
+  <xacro:mesh_link name="base_inertia"
               origin_rpy="0 0 ${pi/2}" origin_xyz="-0.16 0.035 -0.045"
               i_rpy="0 0 0" i_xyz="0 0 0"
@@ -427,5 +427,5 @@
 <xacro:frame_joint name="base_base" type="fixed"
                   origin_rpy="0 0 0" origin_xyz="0 0 0"
-                  parent="base_footprint" child="base_link"/>
+                  parent="base_link" child="base_inertia"/>
 <!-- MAIN BODY TO BATTERY -->
 <xacro:frame_joint name="base_battery" type="fixed"

Commit message: added friction on foot links

File: mini_ros/urdf/spot.urdf.xacro (robot description, xacro)
@@ -121,5 +121,5 @@
                     origin_rpy="0 0 0" origin_xyz="${0.2515-0.16} ${0.0044+0.035} ${0.067-0.045}"
                     parent="front_bracket" child="front_left_hip"
-                    effort="1000.0" velocity="0.7"
+                    effort="3.5" velocity="0.7"
                     damping="0.0"
                     friction="0.0"
@@ -142,5 +142,5 @@
                     origin_rpy="0 0 0" origin_xyz="0.0015 0.045 -0.0087"
                     parent="front_left_hip" child="front_left_upper_leg"
-                    effort="1000.0" velocity="0.7"
+                    effort="3.5" velocity="0.7"
                     damping="0.0"
                     friction="0.0"
@@ -163,5 +163,5 @@
                     origin_rpy="0 0 0" origin_xyz="-0.005 0.018 -0.109"
                     parent="front_left_upper_leg" child="front_left_lower_leg"
-                    effort="1000.0" velocity="0.7"
+                    effort="3.5" velocity="0.7"
                     damping="0.0"
                     friction="0.0"
@@ -201,5 +201,5 @@
                     origin_rpy="0 0 0" origin_xyz="${-0.2515+0.115} ${0.0044+0.035} ${0.067-0.045}"
                     parent="back_bracket" child="back_left_hip"
-                    effort="1000.0" velocity="0.7"
+                    effort="3.5" velocity="0.7"
                     damping="0.0"
                     friction="0.0"
@@ -222,5 +222,5 @@
                     origin_rpy="0 0 0" origin_xyz="0.0015 0.045 -0.0087"
                     parent="back_left_hip" child="back_left_upper_leg"
-                    effort="1000.0" velocity="0.7"
+                    effort="3.5" velocity="0.7"
                     damping="0.0"
                     friction="0.0"
@@ -243,5 +243,5 @@
                     origin_rpy="0 0 0" origin_xyz="-0.005 0.018 -0.109"
                     parent="back_left_upper_leg" child="back_left_lower_leg"
-                    effort="1000.0" velocity="0.7"
+                    effort="3.5" velocity="0.7"
                     damping="0.0"
                     friction="0.0"
@@ -281,5 +281,5 @@
                     origin_rpy="0 0 0" origin_xyz="${0.2515-0.16} ${-(0.0044+0.035)} ${0.067-0.045}"
                     parent="front_bracket" child="front_right_hip"
-                    effort="1000.0" velocity="0.7"
+                    effort="3.5" velocity="0.7"
                     damping="0.0"
                     friction="0.0"
@@ -302,5 +302,5 @@
                     origin_rpy="0 0 0" origin_xyz="0.0015 -0.045 -0.0087"
                     parent="front_right_hip" child="front_right_upper_leg"
-                    effort="1000.0" velocity="0.7"
+                    effort="3.5" velocity="0.7"
                     damping="0.0"
                     friction="0.0"
@@ -323,5 +323,5 @@
                     origin_rpy="0 0 0" origin_xyz="-0.005 -0.018 -0.109"
                     parent="front_right_upper_leg" child="front_right_lower_leg"
-                    effort="1000.0" velocity="0.7"
+                    effort="3.5" velocity="0.7"
                     damping="0.0"
                     friction="0.0"
@@ -361,5 +361,5 @@
                     origin_rpy="0 0 0" origin_xyz="${-0.2515+0.115} ${-(0.0044+0.035)} ${0.067-0.045}"
                     parent="back_bracket" child="back_right_hip"
-                    effort="1000.0" velocity="0.7"
+                    effort="3.5" velocity="0.7"
                     damping="0.0"
                     friction="0.0"
@@ -382,5 +382,5 @@
                     origin_rpy="0 0 0" origin_xyz="0.0015 -0.045 -0.0087"
                     parent="back_right_hip" child="back_right_upper_leg"
-                    effort="1000.0" velocity="0.7"
+                    effort="3.5" velocity="0.7"
                     damping="0.0"
                     friction="0.0"
@@ -403,5 +403,5 @@
                     origin_rpy="0 0 0" origin_xyz="-0.005 -0.018 -0.109"
                     parent="back_right_upper_leg" child="back_right_lower_leg"
-                    effort="1000.0" velocity="0.7"
+                    effort="3.5" velocity="0.7"
                     damping="0.0"
                     friction="0.0"
@@ -466,3 +466,39 @@
 	</plugin>
 </gazebo>
+<gazebo reference="front_left_foot">
+  <kp>1000000.0</kp>
+  <kd>1.0</kd>
+  <mu1>0.8</mu1>
+  <mu2>0.8</mu2>
+  <maxVel>0.0</maxVel>
+  <minDepth>0.001</minDepth>
+  <material>Gazebo/Orange</material>
+</gazebo>
+<gazebo reference="back_left_foot">
+  <kp>1000000.0</kp>
+  <kd>1.0</kd>
+  <mu1>0.8</mu1>
+  <mu2>0.8</mu2>
+  <maxVel>0.0</maxVel>
+  <minDepth>0.001</minDepth>
+  <material>Gazebo/Orange</material>
+</gazebo>
+<gazebo reference="front_right_foot">
+  <kp>1000000.0</kp>
+  <kd>1.0</kd>
+  <mu1>0.8</mu1>
+  <mu2>0.8</mu2>
+  <maxVel>0.0</maxVel>
+  <minDepth>0.001</minDepth>
+  <material>Gazebo/Orange</material>
+</gazebo>
+<gazebo reference="back_right_foot">
+  <kp>1000000.0</kp>
+  <kd>1.0</kd>
+  <mu1>0.8</mu1>
+  <mu2>0.8</mu2>
+  <maxVel>0.0</maxVel>
+  <minDepth>0.001</minDepth>
+  <material>Gazebo/Orange</material>
+</gazebo>
 </robot>

Commit message: shifted foot friction to macro

File: mini_ros/urdf/spot.urdf.xacro (robot description, xacro)
@@ -466,39 +466,3 @@
 	</plugin>
 </gazebo>
-<gazebo reference="front_left_foot">
-  <kp>1000000.0</kp>
-  <kd>1.0</kd>
-  <mu1>0.8</mu1>
-  <mu2>0.8</mu2>
-  <maxVel>0.0</maxVel>
-  <minDepth>0.001</minDepth>
-  <material>Gazebo/Orange</material>
-</gazebo>
-<gazebo reference="back_left_foot">
-  <kp>1000000.0</kp>
-  <kd>1.0</kd>
-  <mu1>0.8</mu1>
-  <mu2>0.8</mu2>
-  <maxVel>0.0</maxVel>
-  <minDepth>0.001</minDepth>
-  <material>Gazebo/Orange</material>
-</gazebo>
-<gazebo reference="front_right_foot">
-  <kp>1000000.0</kp>
-  <kd>1.0</kd>
-  <mu1>0.8</mu1>
-  <mu2>0.8</mu2>
-  <maxVel>0.0</maxVel>
-  <minDepth>0.001</minDepth>
-  <material>Gazebo/Orange</material>
-</gazebo>
-<gazebo reference="back_right_foot">
-  <kp>1000000.0</kp>
-  <kd>1.0</kd>
-  <mu1>0.8</mu1>
-  <mu2>0.8</mu2>
-  <maxVel>0.0</maxVel>
-  <minDepth>0.001</minDepth>
-  <material>Gazebo/Orange</material>
-</gazebo>
 </robot>

File: mini_ros/urdf/spot_macro.xacro (robot description, xacro)
@@ -79,4 +79,13 @@
       </inertial>
     </link>
+    <gazebo reference="${name}">
+      <kp>1000000.0</kp>
+      <kd>1.0</kd>
+      <mu1>0.8</mu1>
+      <mu2>0.8</mu2>
+      <maxVel>0.0</maxVel>
+      <minDepth>0.001</minDepth>
+      <material>Gazebo/Orange</material>
+    </gazebo>
   </xacro:macro>
   <!-- Left Leg: prefix is front or rear -->
