Commit message: Complete re-design of dog. Troubleshooting pybullet sim

File: spotmicro/util/pybullet_data/assets/urdf/spot.urdf (robot description, URDF)
Before this commit: robot rex, 23 links, 22 joints
Links:
- removed link chassis_front_link
- removed link chassis_rear_link
- removed link front_left_foot_link
- removed link front_left_leg_link
- removed link front_left_leg_link_cover
- removed link front_left_shoulder_link
- removed link front_left_toe_link
- removed link front_right_foot_link
- removed link front_right_leg_link
- removed link front_right_leg_link_cover
- removed link front_right_shoulder_link
- removed link front_right_toe_link
- removed link rear_left_foot_link
- removed link rear_left_leg_link
- removed link rear_left_leg_link_cover
- removed link rear_left_shoulder_link
- removed link rear_left_toe_link
- removed link rear_right_foot_link
- removed link rear_right_leg_link
- removed link rear_right_leg_link_cover
- removed link rear_right_shoulder_link
- removed link rear_right_toe_link
- added link back, mass 0.1; collision box size=0.114 0.075 0.085; visual mesh filename=package://mini_ros/stl/OpenQuadruped/Back.stl scale=1 1 1
- added link back_bracket, mass 0.1; collision box size=0.025 0.075 0.085; visual mesh filename=package://mini_ros/stl/OpenQuadruped/Back_Bracket.stl scale=1 1 1
- added link back_left_foot, mass 0.005; collision sphere radius=0.02; visual mesh filename=package://mini_ros/stl/OpenQuadruped/LEFT_FOOT.stl scale=1 1 1
- added link back_left_hip, mass 0.2; collision box size=0.05 0.065 0.065; visual mesh filename=package://mini_ros/stl/OpenQuadruped/LEFT_HIP.stl scale=1 1 1
- added link back_left_lower_leg, mass 0.05; collision box size=0.035 0.035 0.12; visual mesh filename=package://mini_ros/stl/OpenQuadruped/LEFT_LOWER_LEG.stl scale=1 1 1
- added link back_left_upper_leg, mass 0.13; collision box size=0.035 0.035 0.11; visual mesh filename=package://mini_ros/stl/OpenQuadruped/LEFT_UPPER_LEG.stl scale=1 1 1
- added link back_right_foot, mass 0.005; collision sphere radius=0.02; visual mesh filename=package://mini_ros/stl/OpenQuadruped/RIGHT_FOOT.stl scale=1 1 1
- added link back_right_hip, mass 0.2; collision box size=0.05 0.065 0.065; visual mesh filename=package://mini_ros/stl/OpenQuadruped/RIGHT_HIP.stl scale=1 1 1
- added link back_right_lower_leg, mass 0.05; collision box size=0.035 0.035 0.12; visual mesh filename=package://mini_ros/stl/OpenQuadruped/RIGHT_LOWER_LEG.stl scale=1 1 1
- added link back_right_upper_leg, mass 0.13; collision box size=0.035 0.035 0.11; visual mesh filename=package://mini_ros/stl/OpenQuadruped/RIGHT_UPPER_LEG.stl scale=1 1 1
- added link battery, mass 0.4; collision box size=0.048 0.145 0.026; visual mesh filename=package://mini_ros/stl/OpenQuadruped/Battery.stl scale=1 1 1
- added link chassis_left, mass 0.01; collision box size=0.06 0.15 0.006; visual mesh filename=package://mini_ros/stl/OpenQuadruped/Chassis_Left_Side.stl scale=1 1 1
- added link chassis_right, mass 0.01; collision box size=0.06 0.15 0.006; visual mesh filename=package://mini_ros/stl/OpenQuadruped/Chassis_Right_Side.stl scale=1 1 1
- added link front, mass 0.1; collision box size=0.114 0.045 0.085; visual mesh filename=package://mini_ros/stl/OpenQuadruped/Front.stl scale=1 1 1
- added link front_bracket, mass 0.1; collision box size=0.025 0.075 0.085; visual mesh filename=package://mini_ros/stl/OpenQuadruped/Front_Bracket.stl scale=1 1 1
- added link front_left_foot, mass 0.005; collision sphere radius=0.02; visual mesh filename=package://mini_ros/stl/OpenQuadruped/LEFT_FOOT.stl scale=1 1 1
- added link front_left_hip, mass 0.2; collision box size=0.05 0.065 0.065; visual mesh filename=package://mini_ros/stl/OpenQuadruped/LEFT_HIP.stl scale=1 1 1
- added link front_left_lower_leg, mass 0.05; collision box size=0.035 0.035 0.12; visual mesh filename=package://mini_ros/stl/OpenQuadruped/LEFT_LOWER_LEG.stl scale=1 1 1
- added link front_left_upper_leg, mass 0.13; collision box size=0.035 0.035 0.11; visual mesh filename=package://mini_ros/stl/OpenQuadruped/LEFT_UPPER_LEG.stl scale=1 1 1
- added link front_right_foot, mass 0.005; collision sphere radius=0.02; visual mesh filename=package://mini_ros/stl/OpenQuadruped/RIGHT_FOOT.stl scale=1 1 1
- added link front_right_hip, mass 0.2; collision box size=0.05 0.065 0.065; visual mesh filename=package://mini_ros/stl/OpenQuadruped/RIGHT_HIP.stl scale=1 1 1
- added link front_right_lower_leg, mass 0.05; collision box size=0.035 0.035 0.12; visual mesh filename=package://mini_ros/stl/OpenQuadruped/RIGHT_LOWER_LEG.stl scale=1 1 1
- added link front_right_upper_leg, mass 0.13; collision box size=0.035 0.035 0.11; visual mesh filename=package://mini_ros/stl/OpenQuadruped/RIGHT_UPPER_LEG.stl scale=1 1 1
- link base_link: mass 1.20 -> 0.6; geometry collision box size=0.114 0.2 0.1; visual mesh filename=package://mini_ros/stl/OpenQuadruped/MAINBODY.stl scale=1 1 1
Joints:
- removed joint chassis_base_front
- removed joint chassis_base_rear
- removed joint foot_motor_front_left
- removed joint foot_motor_front_right
- removed joint foot_motor_rear_left
- removed joint foot_motor_rear_right
- removed joint front_left_leg_cover_joint
- removed joint front_left_toe
- removed joint front_right_leg_cover_joint
- removed joint front_right_toe
- removed joint motor_front_left_leg
- removed joint motor_front_left_shoulder
- removed joint motor_front_right_leg
- removed joint motor_front_right_shoulder
- removed joint motor_rear_left_leg
- removed joint motor_rear_left_shoulder
- removed joint motor_rear_right_leg
- removed joint motor_rear_right_shoulder
- removed joint rear_left_leg_cover_joint
- removed joint rear_left_toe
- removed joint rear_right_leg_cover_joint
- removed joint rear_right_toe
- added joint back_left_leg_foot: type fixed, parent back_left_lower_leg, child back_left_foot, origin xyz=0 0 -0.1265 rpy=0 0 0
- added joint back_right_leg_foot: type fixed, parent back_right_lower_leg, child back_right_foot, origin xyz=0 0 -0.1265 rpy=0 0 0
- added joint base_back: type fixed, parent base_link, child back, origin xyz=0 0 0 rpy=0 0 0
- added joint base_back_bracket: type fixed, parent base_link, child back_bracket, origin xyz=0 0 0 rpy=0 0 0
- added joint base_battery: type fixed, parent base_link, child battery, origin xyz=-0.01 0 -0.0225 rpy=0 0 0
- added joint base_front: type fixed, parent base_link, child front, origin xyz=0 0 0 rpy=0 0 0
- added joint base_front_bracket: type fixed, parent base_link, child front_bracket, origin xyz=0 0 0 rpy=0 0 0
- added joint base_left: type fixed, parent base_link, child chassis_left, origin xyz=0.00 0.052 0 rpy=0 0 0
- added joint base_right: type fixed, parent base_link, child chassis_right, origin xyz=0.00 -0.052 0 rpy=0 0 0
- added joint front_left_leg_foot: type fixed, parent front_left_lower_leg, child front_left_foot, origin xyz=0 0 -0.1265 rpy=0 0 0
- added joint front_right_leg_foot: type fixed, parent front_right_lower_leg, child front_right_foot, origin xyz=0 0 -0.1265 rpy=0 0 0
- added joint motor_back_left_hip: type revolute, parent back_bracket, child back_left_hip, origin xyz=-0.1365 0.0394 0.022 rpy=0 0 0, axis 1 0 0, limit lower=-1.04 upper=1.04 effort=1000.0 velocity=0.7
- added joint motor_back_left_lower_leg: type revolute, parent back_left_upper_leg, child back_left_lower_leg, origin xyz=-0.005 0.018 -0.109 rpy=0 0 0, axis 0 1 0, limit lower=-2.9 upper=1.57079632679 effort=1000.0 velocity=0.7
- added joint motor_back_left_upper_leg: type revolute, parent back_left_hip, child back_left_upper_leg, origin xyz=0.0015 0.045 -0.0087 rpy=0 0 0, axis 0 1 0, limit lower=-1.57079632679 upper=2.59 effort=1000.0 velocity=0.7
- added joint motor_back_right_hip: type revolute, parent back_bracket, child back_right_hip, origin xyz=-0.1365 -0.0394 0.022 rpy=0 0 0, axis 1 0 0, limit lower=-1.04 upper=1.04 effort=1000.0 velocity=0.7
- added joint motor_back_right_lower_leg: type revolute, parent back_right_upper_leg, child back_right_lower_leg, origin xyz=-0.005 -0.018 -0.109 rpy=0 0 0, axis 0 1 0, limit lower=-2.9 upper=1.57079632679 effort=1000.0 velocity=0.7
- added joint motor_back_right_upper_leg: type revolute, parent back_right_hip, child back_right_upper_leg, origin xyz=0.0015 -0.045 -0.0087 rpy=0 0 0, axis 0 1 0, limit lower=-1.57079632679 upper=2.59 effort=1000.0 velocity=0.7
- added joint motor_front_left_hip: type revolute, parent front_bracket, child front_left_hip, origin xyz=0.0915 0.0394 0.022 rpy=0 0 0, axis 1 0 0, limit lower=-1.04 upper=1.04 effort=1000.0 velocity=0.7
- added joint motor_front_left_lower_leg: type revolute, parent front_left_upper_leg, child front_left_lower_leg, origin xyz=-0.005 0.018 -0.109 rpy=0 0 0, axis 0 1 0, limit lower=-2.9 upper=1.57079632679 effort=1000.0 velocity=0.7
- added joint motor_front_left_upper_leg: type revolute, parent front_left_hip, child front_left_upper_leg, origin xyz=0.0015 0.045 -0.0087 rpy=0 0 0, axis 0 1 0, limit lower=-1.57079632679 upper=2.59 effort=1000.0 velocity=0.7
- added joint motor_front_right_hip: type revolute, parent front_bracket, child front_right_hip, origin xyz=0.0915 -0.0394 0.022 rpy=0 0 0, axis 1 0 0, limit lower=-1.04 upper=1.04 effort=1000.0 velocity=0.7
- added joint motor_front_right_lower_leg: type revolute, parent front_right_upper_leg, child front_right_lower_leg, origin xyz=-0.005 -0.018 -0.109 rpy=0 0 0, axis 0 1 0, limit lower=-2.9 upper=1.57079632679 effort=1000.0 velocity=0.7
- added joint motor_front_right_upper_leg: type revolute, parent front_right_hip, child front_right_upper_leg, origin xyz=0.0015 -0.045 -0.0087 rpy=0 0 0, axis 0 1 0, limit lower=-1.57079632679 upper=2.59 effort=1000.0 velocity=0.7

Commit message: visual issue seems to have spread to heightfield generator

File: mini_ros/urdf/spot.urdf (robot description, URDF)
Before this commit: robot spot, 25 links, 24 joints
Links:
- link back_left_foot: geometry collision mesh filename=package://mini_ros/stl/OpenQuadruped/LEFT_FOOT.stl scale=1 1 1; visual mesh filename=package://mini_ros/stl/OpenQuadruped/LEFT_FOOT.stl scale=1 1 1
- link back_right_foot: geometry collision mesh filename=package://mini_ros/stl/OpenQuadruped/RIGHT_FOOT.stl scale=1 1 1; visual mesh filename=package://mini_ros/stl/OpenQuadruped/RIGHT_FOOT.stl scale=1 1 1
- link front_left_foot: geometry collision mesh filename=package://mini_ros/stl/OpenQuadruped/LEFT_FOOT.stl scale=1 1 1; visual mesh filename=package://mini_ros/stl/OpenQuadruped/LEFT_FOOT.stl scale=1 1 1
- link front_right_foot: geometry collision mesh filename=package://mini_ros/stl/OpenQuadruped/RIGHT_FOOT.stl scale=1 1 1; visual mesh filename=package://mini_ros/stl/OpenQuadruped/RIGHT_FOOT.stl scale=1 1 1

File: mini_ros/urdf/spot.urdf.xacro (robot description, xacro)
@@ -172,5 +172,5 @@
               i_rpy="0 0 0" i_xyz="0 0 0"
               mass="0.005"
-              c_xyz="-0.005 0 0"
+              c_xyz="${-0.247} ${-0.068} ${0.18}"
               length="0.05"
               width="0.065"
@@ -252,5 +252,5 @@
               i_rpy="0 0 0" i_xyz="0 0 0"
               mass="0.005"
-              c_xyz="-0.005 0 0"
+              c_xyz="${-0.247} ${-0.068} ${0.18}"
               length="0.05"
               width="0.065"
@@ -332,5 +332,5 @@
               i_rpy="0 0 0" i_xyz="0 0 0"
               mass="0.005"
-              c_xyz="-0.005 0 0"
+              c_xyz="${-0.247} ${0.138} ${0.18}"
               length="0.05"
               width="0.065"
@@ -412,5 +412,5 @@
               i_rpy="0 0 0" i_xyz="0 0 0"
               mass="0.005"
-              c_xyz="-0.005 0 0"
+              c_xyz="${-0.247} ${0.138} ${0.18}"
               length="0.05"
               width="0.065"

File: spotmicro/util/pybullet_data/assets/urdf/spot.urdf (robot description, URDF)
Before this commit: robot spot, 24 links, 23 joints
Links:
- link back: geometry collision box size=0.114 0.075 0.085; visual mesh filename=package://mini_ros/stl/OpenQuadruped/Back.stl scale=1 1 1
- link back_bracket: geometry collision box size=0.025 0.075 0.085; visual mesh filename=package://mini_ros/stl/OpenQuadruped/Back_Bracket.stl scale=1 1 1
- link back_left_foot: geometry collision mesh filename=package://mini_ros/stl/OpenQuadruped/LEFT_FOOT.stl scale=1 1 1; visual mesh filename=package://mini_ros/stl/OpenQuadruped/LEFT_FOOT.stl scale=1 1 1
- link back_left_hip: geometry collision box size=0.05 0.065 0.065; visual mesh filename=package://mini_ros/stl/OpenQuadruped/LEFT_HIP.stl scale=1 1 1
- link back_left_lower_leg: geometry collision box size=0.035 0.035 0.12; visual mesh filename=package://mini_ros/stl/OpenQuadruped/LEFT_LOWER_LEG.stl scale=1 1 1
- link back_left_upper_leg: geometry collision box size=0.035 0.035 0.11; visual mesh filename=package://mini_ros/stl/OpenQuadruped/LEFT_UPPER_LEG.stl scale=1 1 1
- link back_right_foot: geometry collision mesh filename=package://mini_ros/stl/OpenQuadruped/RIGHT_FOOT.stl scale=1 1 1; visual mesh filename=package://mini_ros/stl/OpenQuadruped/RIGHT_FOOT.stl scale=1 1 1
- link back_right_hip: geometry collision box size=0.05 0.065 0.065; visual mesh filename=package://mini_ros/stl/OpenQuadruped/RIGHT_HIP.stl scale=1 1 1
- link back_right_lower_leg: geometry collision box size=0.035 0.035 0.12; visual mesh filename=package://mini_ros/stl/OpenQuadruped/RIGHT_LOWER_LEG.stl scale=1 1 1
- link back_right_upper_leg: geometry collision box size=0.035 0.035 0.11; visual mesh filename=package://mini_ros/stl/OpenQuadruped/RIGHT_UPPER_LEG.stl scale=1 1 1
- link base_link: geometry collision box size=0.114 0.2 0.1; visual mesh filename=package://mini_ros/stl/OpenQuadruped/MAINBODY.stl scale=1 1 1
- link battery: geometry collision box size=0.048 0.145 0.026; visual mesh filename=package://mini_ros/stl/OpenQuadruped/Battery.stl scale=1 1 1
- link chassis_left: geometry collision box size=0.06 0.15 0.006; visual mesh filename=package://mini_ros/stl/OpenQuadruped/Chassis_Left_Side.stl scale=1 1 1
- link chassis_right: geometry collision box size=0.06 0.15 0.006; visual mesh filename=package://mini_ros/stl/OpenQuadruped/Chassis_Right_Side.stl scale=1 1 1
- link front: geometry collision box size=0.114 0.045 0.085; visual mesh filename=package://mini_ros/stl/OpenQuadruped/Front.stl scale=1 1 1
- link front_bracket: geometry collision box size=0.025 0.075 0.085; visual mesh filename=package://mini_ros/stl/OpenQuadruped/Front_Bracket.stl scale=1 1 1
- link front_left_foot: geometry collision mesh filename=package://mini_ros/stl/OpenQuadruped/LEFT_FOOT.stl scale=1 1 1; visual mesh filename=package://mini_ros/stl/OpenQuadruped/LEFT_FOOT.stl scale=1 1 1
- link front_left_hip: geometry collision box size=0.05 0.065 0.065; visual mesh filename=package://mini_ros/stl/OpenQuadruped/LEFT_HIP.stl scale=1 1 1
- link front_left_lower_leg: geometry collision box size=0.035 0.035 0.12; visual mesh filename=package://mini_ros/stl/OpenQuadruped/LEFT_LOWER_LEG.stl scale=1 1 1
- link front_left_upper_leg: geometry collision box size=0.035 0.035 0.11; visual mesh filename=package://mini_ros/stl/OpenQuadruped/LEFT_UPPER_LEG.stl scale=1 1 1
- link front_right_foot: geometry collision mesh filename=package://mini_ros/stl/OpenQuadruped/RIGHT_FOOT.stl scale=1 1 1; visual mesh filename=package://mini_ros/stl/OpenQuadruped/RIGHT_FOOT.stl scale=1 1 1
- link front_right_hip: geometry collision box size=0.05 0.065 0.065; visual mesh filename=package://mini_ros/stl/OpenQuadruped/RIGHT_HIP.stl scale=1 1 1
- link front_right_lower_leg: geometry collision box size=0.035 0.035 0.12; visual mesh filename=package://mini_ros/stl/OpenQuadruped/RIGHT_LOWER_LEG.stl scale=1 1 1
- link front_right_upper_leg: geometry collision box size=0.035 0.035 0.11; visual mesh filename=package://mini_ros/stl/OpenQuadruped/RIGHT_UPPER_LEG.stl scale=1 1 1

Commit message: generate new urdf

File: mini_ros/urdf/spot.urdf (robot description, URDF)
Before this commit: robot spot, 25 links, 24 joints
Links:
- removed link base_footprint
- added link base_inertia, mass 0.6; collision box size=0.114 0.2 0.1; visual mesh filename=package://mini_ros/stl/OpenQuadruped/MAINBODY.stl scale=1 1 1
- link base_link: mass 0.6 -> None; geometry 
Joints:
- joint base_base: child base_link -> base_inertia; parent base_footprint -> base_link
- joint motor_back_left_hip: limit lower=-1.04 upper=1.04 effort=1000.0 velocity=0.7 -> lower=-1.04 upper=1.04 effort=4.0 velocity=4.0
- joint motor_back_left_lower_leg: limit lower=-2.9 upper=1.57079632679 effort=1000.0 velocity=0.7 -> lower=-2.9 upper=1.57079632679 effort=4.0 velocity=4.0
- joint motor_back_left_upper_leg: limit lower=-1.57079632679 upper=2.59 effort=1000.0 velocity=0.7 -> lower=-1.57079632679 upper=2.59 effort=4.0 velocity=4.0
- joint motor_back_right_hip: limit lower=-1.04 upper=1.04 effort=1000.0 velocity=0.7 -> lower=-1.04 upper=1.04 effort=4.0 velocity=4.0
- joint motor_back_right_lower_leg: limit lower=-2.9 upper=1.57079632679 effort=1000.0 velocity=0.7 -> lower=-2.9 upper=1.57079632679 effort=4.0 velocity=4.0
- joint motor_back_right_upper_leg: limit lower=-1.57079632679 upper=2.59 effort=1000.0 velocity=0.7 -> lower=-1.57079632679 upper=2.59 effort=4.0 velocity=4.0
- joint motor_front_left_hip: limit lower=-1.04 upper=1.04 effort=1000.0 velocity=0.7 -> lower=-1.04 upper=1.04 effort=4.0 velocity=4.0
- joint motor_front_left_lower_leg: limit lower=-2.9 upper=1.57079632679 effort=1000.0 velocity=0.7 -> lower=-2.9 upper=1.57079632679 effort=4.0 velocity=4.0
- joint motor_front_left_upper_leg: limit lower=-1.57079632679 upper=2.59 effort=1000.0 velocity=0.7 -> lower=-1.57079632679 upper=2.59 effort=4.0 velocity=4.0
- joint motor_front_right_hip: limit lower=-1.04 upper=1.04 effort=1000.0 velocity=0.7 -> lower=-1.04 upper=1.04 effort=4.0 velocity=4.0
- joint motor_front_right_lower_leg: limit lower=-2.9 upper=1.57079632679 effort=1000.0 velocity=0.7 -> lower=-2.9 upper=1.57079632679 effort=4.0 velocity=4.0
- joint motor_front_right_upper_leg: limit lower=-1.57079632679 upper=2.59 effort=1000.0 velocity=0.7 -> lower=-1.57079632679 upper=2.59 effort=4.0 velocity=4.0

File: mini_ros/urdf/spot.urdf.xacro (robot description, xacro)
@@ -4,5 +4,5 @@
   <xacro:include filename="$(find mini_ros)/urdf/spot_macro.xacro" />
   <xacro:include filename="$(find mini_ros)/urdf/transmissions.xacro" />
-  <xacro:include filename="$(find mini_ros)/urdf/accessories.urdf.xacro" />
+  <!-- <xacro:include filename="$(find mini_ros)/urdf/accessories.urdf.xacro" /> -->
   <!-- Robot description -->
   <!-- STATIC Links -->
